Commit message: navstack tutorial code

File: src/robot_description/models/mariam_agent.urdf (robot description, URDF)
Before this commit: robot mariam_agent, 4 links, 3 joints
Links:
- added link lidar_link, mass 0.114; collision cylinder length=0.18 radius=0.0508; visual cylinder length=0.18 radius=0.0508
Joints:
- added joint lidar_joint: type fixed, parent base_link, child lidar_link, origin xyz=0 0 0.13 rpy=0 0 0
