Commit message: URDF model significantly improved. Packages mariam_description and mariam_navigation have major changes and different organization.

File: src/mariam_description/gazebo_models/basic_mobile_bot_description/model.urdf (robot description, URDF)
Before this commit: robot mariam, 3 links, 2 joints
Links:
- removed link camera_link
- added link front_caster; collision sphere radius=${(wheel_radius+wheel_zoff-(base_height/2))}; visual sphere radius=${(wheel_radius+wheel_zoff-(base_height/2))}
- added link gps_link
- added link imu_link
- added link lidar_link, mass 0.114; collision cylinder length=0.18 radius=0.0508; visual cylinder length=0.18 radius=0.0508
Joints:
- removed joint camera_joint
- added joint caster_joint: type fixed, parent base_link, child front_caster, origin xyz=${caster_xoff} 0.0 ${-(base_height/2)} rpy=0 0 0
- added joint gps_joint: type fixed, parent base_link, child gps_link, origin xyz=0.10 0 0.05 rpy=0 0 0
- added joint imu_joint: type fixed, parent base_link, child imu_link, origin xyz=-0.10 0 0.05 rpy=0 0 0
- added joint lidar_joint: type fixed, parent base_link, child lidar_link, origin xyz=0.215 0 0.13 rpy=0 0 0

File: src/mariam_description/xacro_models/mariam.urdf.xacro (robot description, xacro)
@@ -47,6 +47,7 @@
     <origin xyz="0.0 0.0 ${(wheel_radius+wheel_zoff)}" rpy="0 0 0"/>
   </joint>
-  <!-- ********************** ROBOT BASE *********************************  -->
+  <!-- ********************** ROBOT CHASSIS *********************************  -->
   <link name="base_link">
+    <!-- base chassis -->
     <visual>
       <origin xyz="0 0 0" rpy="0 0 0"/>
@@ -63,9 +64,38 @@
       </geometry>
     </collision>
+    <!-- computer -->
+    <visual>
+      <origin xyz="-0.01 0 ${base_height/2 + 0.05}" rpy="0 0 0"/>
+      <geometry>
+        <box size="${base_length - 0.08} ${base_width - 0.06} 0.1"/>
+      </geometry>
+      <material name="Red">
+        <color rgba="${255/255} ${0/255} ${0/255} 1.0"/>
+      </material>
+    </visual>
+    <collision>
+      <origin xyz="-0.01 0 ${base_height/2 + 0.05}" rpy="0 0 0"/>
+      <geometry>
+        <box size="${base_length - 0.08} ${base_width - 0.06} 0.1"/>
+      </geometry>
+    </collision>
+    <!-- camera stand -->
+    <visual>
+      <origin xyz="-${(base_length/2) + 0.01} 0 ${((0.3 - (0.027/2)) - base_height/2)/2}" rpy="0 0 0"/>
+      <geometry>
+        <box size="0.02 0.02 ${0.3 - (0.027/2) + base_height/2}"/>
+      </geometry>
+      <material name="Red">
+        <color rgba="${255/255} ${0/255} ${0/255} 1.0"/>
+      </material>
+    </visual>
+    <collision>
+      <origin xyz="-${(base_length/2) + 0.01} 0 ${((0.3 - (0.027/2)) - base_height/2)/2}" rpy="0 0 0"/>
+      <geometry>
+        <box size="0.02 0.02 ${0.3 - (0.027/2) + base_height/2}"/>
+      </geometry>
+    </collision>
     <xacro:box_inertia m="40.0" w="${base_width}" d="${base_length}" h="${base_height}"/>
   </link>
-  <gazebo reference="base_link">
-    <material>Gazebo/Red</material>
-  </gazebo>
   <!-- *********************** DRIVE WHEELS ******************************  -->
   <xacro:macro name="wheel" params="prefix x_reflect y_reflect">
@@ -86,15 +116,16 @@
         </geometry>
       </collision>
-      <xacro:cylinder_inertia m="20.0" r="${wheel_radius}" h="${wheel_width}"/>
+      <xacro:cylinder_inertia m="5.0" r="${wheel_radius}" h="${wheel_width}"/>
     </link>
     <!-- Connect the wheels to the base_link at the appropriate location, and
          define a continuous joint to allow the wheels to freely rotate about
          an axis -->
-    <joint name="${prefix}_joint" type="revolute">
+    <joint name="${prefix}_joint" type="continuous">
       <parent link="base_link"/>
       <child link="${prefix}_link"/>
       <origin xyz="${x_reflect*wheel_xoff} ${y_reflect*(base_width/2+wheel_ygap)} ${-wheel_zoff}" rpy="0 0 0"/>
-      <limit upper="3.1415" lower="-3.1415" effort="30" velocity="5.0"/>
       <axis xyz="0 1 0"/>
+      <!-- <limit effort="10000" velocity="1000"/> -->
+      <dynamics damping="0.5" friction="0.1"/>
     </joint>
   </xacro:macro>
@@ -126,6 +157,8 @@
     <parent link="base_link"/>
     <child link="camera_link"/>
-    <origin xyz="-${base_length/2} 0 0.3" rpy="0 0 0"/>
+    <origin xyz="-${base_length/2 + 0.01} 0 0.3" rpy="0 0 0"/>
   </joint>
+  <!-- *********************** GAZEBO SETUP **********************************  -->
+  <xacro:include filename="$(find mariam_description)/xacro_models/mariam_gazebo.urdf.xacro"/>
   <!-- *********************** INTERBOTIX SETUP **********************************  -->
   <!-- Include the robotic arm xacro file -->
