Commit message: updated xacro files and urdf launch file

File: src/mariam_description/xacro_models/mariam.urdf.xacro (robot description, xacro)
@@ -172,12 +172,14 @@
   </joint> -->
   <!-- *********************** MODIFIED INTERBOTIX SETUP **********************************  -->
-  <!-- Include the robotic arm xacro file -->
-  <!-- <xacro:include filename="$(find mariam_description)/models/px100_original.urdf.xacro" />
-   -->
-  <!-- Attach the robotic arm to the base_link -->
-  <!-- <joint name="arm_base_joint" type="fixed">
+    <!-- Attach the robotic arm to the base_link -->
+  <joint name="arm_base_joint" type="fixed">
     <parent link="base_link"/>
     <child link="px100/base_link"/>
-    <origin xyz="${base_length/1.5} 0 ${base_height/2}" rpy="0 0 -${pi/2}"/>
-  </joint> -->
+    <!-- <origin xyz="${base_length/1.5} 0 ${base_height/2}" rpy="0 0 -${pi/2}"/> -->
+    <origin
+        rpy="0 0 ${pi/2}"
+        xyz="0 0 0" />
+  </joint>
+  <!-- Include the robotic arm xacro file -->
+  <xacro:include filename="$(find mariam_description)/xacro_models/px100_modified.urdf.xacro" />
 </robot>

File: src/mariam_description/xacro_models/mariam_gazebo.urdf.xacro (robot description, xacro)
@@ -172,8 +172,8 @@
   </gazebo>
   <!-- *********************** GAZEBO ROS CONTROL *********************   -->
-  <!-- <gazebo>
+  <gazebo>
     <plugin name="gazebo_ros_control" filename="libgazebo_ros_control.so">
       <robotNamespace>/</robotNamespace>
     </plugin>
-  </gazebo> -->
+  </gazebo>
 </robot>

File: src/mariam_description/xacro_models/px100_modified.urdf.xacro (robot description, xacro)
@@ -7,5 +7,5 @@
     value="4"
     scope="global" />
-  <xacro:arg name="robot_name" default="${robot_model}" />
+  <xacro:arg name="robot_name" default="" />
   <xacro:arg name="base_link_frame" default="base_link" />
   <xacro:arg name="use_gripper" default="false" /> <!-- Modified from true -->
@@ -45,4 +45,7 @@
     <texture filename="package://interbotix_xsarm_descriptions/meshes/interbotix_black.png" />
   </material>
+  <material name="my_pink">
+        <color rgba="1 0.4 0.7 1.0" />  <!-- Pink color (R=1, G=0.4, B=0.7, fully opaque) -->
+  </material>
   <xacro:if value="$(arg use_world_frame)">
     <link name="world" />
@@ -65,5 +68,5 @@
           scale="0.001 0.001 0.001" />
       </geometry>
-      <material name="interbotix_black" />
+      <material name="my_pink" />
     </visual>
     <collision>
@@ -119,5 +122,5 @@
           scale="0.001 0.001 0.001" />
       </geometry>
-      <material name="interbotix_black" />
+      <material name="my_pink" />
     </visual>
     <collision>
@@ -173,5 +176,5 @@
           scale="0.001 0.001 0.001" />
       </geometry>
-      <material name="interbotix_black" />
+      <material name="my_pink" />
     </visual>
     <collision>
@@ -227,5 +230,5 @@
           scale="0.001 0.001 0.001" />
       </geometry>
-      <material name="interbotix_black" />
+      <material name="my_pink" />
     </visual>
     <collision>
@@ -359,5 +362,5 @@
             scale="0.001 0.001 0.001" />
         </geometry>
-        <material name="interbotix_black" />
+        <material name="my_pink" />
       </visual>
       <collision>
@@ -412,5 +415,5 @@
               scale="0.001 0.001 0.001" />
           </geometry>
-          <material name="interbotix_black" />
+          <material name="my_pink" />
         </visual>
         <collision>
@@ -490,5 +493,5 @@
                 scale="0.001 0.001 0.001" />
             </geometry>
-            <material name="interbotix_black" />
+            <material name="my_pink" />
           </visual>
           <collision>
@@ -550,5 +553,5 @@
                 scale="0.001 0.001 0.001" />
             </geometry>
-            <material name="interbotix_black" />
+            <material name="my_pink" />
           </visual>
           <collision>

Commit message: updated px100_modified.urdf.xacro, added modified px100 in mariam.urdf.xacro, added rqt steering and camera node to mariam_gazebo.launch.py

File: src/mariam_description/xacro_models/mariam.urdf.xacro (robot description, xacro)
@@ -176,8 +176,8 @@
     <parent link="base_link"/>
     <child link="px100/base_link"/>
-    <!-- <origin xyz="${base_length/1.5} 0 ${base_height/2}" rpy="0 0 -${pi/2}"/> -->
-    <origin
-        rpy="0 0 ${pi/2}"
-        xyz="0 0 0" />
+    <origin xyz="${base_length/1.5} 0 ${base_height/2}" rpy="0 0 -${pi/2}"/>
+    <!-- <origin -->
+        <!-- rpy="0 0 ${pi/2}" -->
+        <!-- xyz="0 0 0" /> -->
   </joint>
   <!-- Include the robotic arm xacro file -->

File: src/mariam_description/xacro_models/px100_modified.urdf.xacro (robot description, xacro)
@@ -7,5 +7,5 @@
     value="4"
     scope="global" />
-  <xacro:arg name="robot_name" default="" />
+  <xacro:arg name="robot_name" default="px100" />
   <xacro:arg name="base_link_frame" default="base_link" />
   <xacro:arg name="use_gripper" default="false" /> <!-- Modified from true -->
@@ -45,5 +45,5 @@
     <texture filename="package://interbotix_xsarm_descriptions/meshes/interbotix_black.png" />
   </material>
-  <material name="my_pink">
+  <material name="gripper_pink">
         <color rgba="1 0.4 0.7 1.0" />  <!-- Pink color (R=1, G=0.4, B=0.7, fully opaque) -->
   </material>
@@ -68,5 +68,5 @@
           scale="0.001 0.001 0.001" />
       </geometry>
-      <material name="my_pink" />
+      <material name="interbotix_black" />
     </visual>
     <collision>
@@ -122,5 +122,5 @@
           scale="0.001 0.001 0.001" />
       </geometry>
-      <material name="my_pink" />
+      <material name="interbotix_black" />
     </visual>
     <collision>
@@ -176,5 +176,5 @@
           scale="0.001 0.001 0.001" />
       </geometry>
-      <material name="my_pink" />
+      <material name="interbotix_black" />
     </visual>
     <collision>
@@ -230,5 +230,5 @@
           scale="0.001 0.001 0.001" />
       </geometry>
-      <material name="my_pink" />
+      <material name="interbotix_black" />
     </visual>
     <collision>
@@ -284,7 +284,5 @@
           scale="0.001 0.001 0.001" />
       </geometry>
-      <material name="pink_material">
-        <color rgba="1 0.4 0.7 1.0" />  <!-- Pink color (R=1, G=0.4, B=0.7, fully opaque) -->
-      </material>
+      <material name="gripper_pink" />
     </visual>
     <collision>
@@ -362,5 +360,5 @@
             scale="0.001 0.001 0.001" />
         </geometry>
-        <material name="my_pink" />
+        <material name="interbotix_black" />
       </visual>
       <collision>
@@ -415,5 +413,5 @@
               scale="0.001 0.001 0.001" />
           </geometry>
-          <material name="my_pink" />
+          <material name="interbotix_black" />
         </visual>
         <collision>
@@ -493,5 +491,5 @@
                 scale="0.001 0.001 0.001" />
             </geometry>
-            <material name="my_pink" />
+            <material name="interbotix_black" />
           </visual>
           <collision>
@@ -553,5 +551,5 @@
                 scale="0.001 0.001 0.001" />
             </geometry>
-            <material name="my_pink" />
+            <material name="interbotix_black" />
           </visual>
           <collision>
@@ -607,5 +605,5 @@
   </xacro:if> <!--
   use_gripper -->
-  <xacro:include filename="$(find interbotix_xsarm_descriptions)/urdf/control.urdf.xacro" />
+  <!-- <xacro:include filename="$(find interbotix_xsarm_descriptions)/urdf/control.urdf.xacro" /> -->
   <xacro:include filename="$(find interbotix_xsarm_descriptions)/urdf/gazebo_configs.urdf.xacro" />
   <xacro:if value="${hardware_type == 'gz_classic'}">

Commit message: updated namespace for px100_modified; added arm controller and joint state broadcaster to mariam_gazebo.launch.py

File: src/mariam_description/xacro_models/mariam.urdf.xacro (robot description, xacro)
@@ -2,4 +2,5 @@
 <robot name="mariam" xmlns:xacro="http://ros.org/wiki/xacro">
   <!-- ****************** ROBOT CONSTANTS *******************************  -->
+  <xacro:arg name="robot_name" default="mariam"/>
   <!-- Define the size of the robot's main chassis in meters -->
   <xacro:property name="base_width" value="0.20"/>
@@ -175,5 +176,5 @@
   <joint name="arm_base_joint" type="fixed">
     <parent link="base_link"/>
-    <child link="px100/base_link"/>
+    <child link="$(arg robot_name)/px100_base_link"/>
     <origin xyz="${base_length/1.5} 0 ${base_height/2}" rpy="0 0 -${pi/2}"/>
     <!-- <origin -->

File: src/mariam_description/xacro_models/mariam_gazebo.urdf.xacro (robot description, xacro)
@@ -173,5 +173,5 @@
   <!-- *********************** GAZEBO ROS CONTROL *********************   -->
   <gazebo>
-    <plugin name="gazebo_ros_control" filename="libgazebo_ros_control.so">
+    <plugin name="mariam_gazebo_ros_control" filename="libgazebo_ros_control.so">
       <robotNamespace>/</robotNamespace>
     </plugin>

File: src/mariam_description/xacro_models/px100_modified.urdf.xacro (robot description, xacro)
@@ -7,10 +7,10 @@
     value="4"
     scope="global" />
-  <xacro:arg name="robot_name" default="px100" />
-  <xacro:arg name="base_link_frame" default="base_link" />
+  <!-- <xacro:arg name="robot_name" default="px100" /> -->
+  <xacro:arg name="base_link_frame" default="px100_base_link" />
   <xacro:arg name="use_gripper" default="false" /> <!-- Modified from true -->
   <xacro:arg name="show_ar_tag" default="false" />
-  <xacro:arg name="show_gripper_bar" default="true" />
-  <xacro:arg name="show_gripper_fingers" default="true" />
+  <xacro:arg name="show_gripper_bar" default="false" />
+  <xacro:arg name="show_gripper_fingers" default="false" />
   <xacro:arg name="use_world_frame" default="false" />
   <xacro:arg name="external_urdf_loc" default="" />

Commit message: set up urdf files and mariam_gazebo.launch.py to launch more than one robot

File: src/mariam_description/xacro_models/mariam.urdf.xacro (robot description, xacro)
@@ -176,5 +176,5 @@
   <joint name="arm_base_joint" type="fixed">
     <parent link="base_link"/>
-    <child link="$(arg robot_name)/px100_base_link"/>
+    <child link="px100/px100_base_link"/>
     <origin xyz="${base_length/1.5} 0 ${base_height/2}" rpy="0 0 -${pi/2}"/>
     <!-- <origin -->

File: src/mariam_description/xacro_models/mariam_gazebo.urdf.xacro (robot description, xacro)
@@ -52,4 +52,5 @@
       <odometry_source>0</odometry_source>
       <ros>
+        <namespace>/$(arg robot_name)</namespace>
         <remapping>odom:=wheel/odometry</remapping>
       </ros>
@@ -60,4 +61,5 @@
     <plugin name="mariam_agent_joint_state" filename="libgazebo_ros_joint_state_publisher.so">
       <ros>
+        <namespace>/$(arg robot_name)</namespace>
         <remapping>~/out:=joint_states</remapping>
       </ros>
@@ -87,4 +89,7 @@
       </camera>
       <plugin name="camera_controller" filename="libgazebo_ros_camera.so">
+        <ros>
+          <namespace>/$(arg robot_name)</namespace>
+        </ros>
         <always_on>true</always_on>
         <update_rate>30.0</update_rate>
@@ -165,5 +170,5 @@
         <frame_name>camera_link</frame_name>
         <ros>
-          <namespace>/imu</namespace>
+          <namespace>/$(arg robot_name)/imu</namespace>
           <remapping>~/out:=data</remapping>
         </ros>
@@ -192,5 +197,9 @@
         <measure_direction>parent_to_child</measure_direction>
       </force_torque>
-      <plugin name="ForceSensorPlugin" filename="libforce_sensor.so"/>
+      <plugin name="ForceSensorPlugin" filename="libforce_sensor.so">
+        <ros>
+          <namespace>/$(arg robot_name)</namespace>
+        </ros>
+      </plugin>
     </sensor>
   </gazebo>

File: src/mariam_description/xacro_models/px100_modified.urdf.xacro (robot description, xacro)
@@ -7,5 +7,5 @@
     value="4"
     scope="global" />
-  <!-- <xacro:arg name="robot_name" default="px100" /> -->
+  <xacro:arg name="arm_name" default="px100" />
   <xacro:arg name="base_link_frame" default="px100_base_link" />
   <xacro:arg name="use_gripper" default="false" /> <!-- Modified from true -->
@@ -54,9 +54,9 @@
         link="world" />
       <child
-        link="$(arg robot_name)/$(arg base_link_frame)" />
+        link="$(arg arm_name)/$(arg base_link_frame)" />
     </joint>
   </xacro:if> <!--
   use_world_frame -->
-  <link name="$(arg robot_name)/$(arg base_link_frame)">
+  <link name="$(arg arm_name)/$(arg base_link_frame)">
     <visual>
       <origin
@@ -105,12 +105,12 @@
       xyz="0 0 0.05085" />
     <parent
-      link="$(arg robot_name)/$(arg base_link_frame)" />
+      link="$(arg arm_name)/$(arg base_link_frame)" />
     <child
-      link="$(arg robot_name)/shoulder_link" />
+      link="$(arg arm_name)/shoulder_link" />
     <dynamics
       friction="0.1"
       damping="0.1" />
   </joint>
-  <link name="$(arg robot_name)/shoulder_link">
+  <link name="$(arg arm_name)/shoulder_link">
     <visual>
       <origin
@@ -159,12 +159,12 @@
       xyz="0 0 0.04225" />
     <parent
-      link="$(arg robot_name)/shoulder_link" />
+      link="$(arg arm_name)/shoulder_link" />
     <child
-      link="$(arg robot_name)/upper_arm_link" />
+      link="$(arg arm_name)/upper_arm_link" />
     <dynamics
       friction="0.1"
       damping="0.1" />
   </joint>
-  <link name="$(arg robot_name)/upper_arm_link">
+  <link name="$(arg arm_name)/upper_arm_link">
     <visual>
       <origin
@@ -213,12 +213,12 @@
       xyz="0.035 0 0.1" />
     <parent
-      link="$(arg robot_name)/upper_arm_link" />
+      link="$(arg arm_name)/upper_arm_link" />
     <child
-      link="$(arg robot_name)/forearm_link" />
+      link="$(arg arm_name)/forearm_link" />
     <dynamics
       friction="0.1"
       damping="0.1" />
   </joint>
-  <link name="$(arg robot_name)/forearm_link">
+  <link name="$(arg arm_name)/forearm_link">
     <visual>
       <origin
@@ -267,12 +267,12 @@
       xyz="0.1 0 0" />
     <parent
-      link="$(arg robot_name)/forearm_link" />
+      link="$(arg arm_name)/forearm_link" />
     <child
-      link="$(arg robot_name)/gripper_link" />
+      link="$(arg arm_name)/gripper_link" />
     <dynamics
       friction="0.1"
       damping="0.1" />
   </joint>
-  <link name="$(arg robot_name)/gripper_link">
+  <link name="$(arg arm_name)/gripper_link">
     <visual>
       <origin
@@ -316,9 +316,9 @@
       xyz="0.10 0 0.01" />
     <parent
-      link="$(arg robot_name)/gripper_link" />
+      link="$(arg arm_name)/gripper_link" />
     <child
-      link="$(arg robot_name)/ee_arm_link" />
+      link="$(arg arm_name)/ee_arm_link" />
   </joint>
-  <link name="$(arg robot_name)/ee_arm_link">
+  <link name="$(arg arm_name)/ee_arm_link">
     <inertial>
       <mass value="0.001" />
@@ -343,12 +343,12 @@
         xyz="0.0055 0 0" />
       <parent
-        link="$(arg robot_name)/ee_arm_link" />
+        link="$(arg arm_name)/ee_arm_link" />
       <child
-        link="$(arg robot_name)/gripper_prop_link" />
+        link="$(arg arm_name)/gripper_prop_link" />
       <dynamics
         friction="0.1"
         damping="0.1" />
     </joint>
-    <link name="$(arg robot_name)/gripper_prop_link">
+    <link name="$(arg arm_name)/gripper_prop_link">
       <visual>
         <origin
@@ -399,9 +399,9 @@
           xyz="0 0 0" />
         <parent
-          link="$(arg robot_name)/ee_arm_link" />
+          link="$(arg arm_name)/ee_arm_link" />
         <child
-          link="$(arg robot_name)/gripper_bar_link" />
+          link="$(arg arm_name)/gripper_bar_link" />
       </joint>
-      <link name="$(arg robot_name)/gripper_bar_link">
+      <link name="$(arg arm_name)/gripper_bar_link">
         <visual>
           <origin
@@ -445,9 +445,9 @@
           xyz="0.023 0 0" />
         <parent
-          link="$(arg robot_name)/gripper_bar_link" />
+          link="$(arg arm_name)/gripper_bar_link" />
         <child
-          link="$(arg robot_name)/fingers_link" />
+          link="$(arg arm_name)/fingers_link" />
       </joint>
-      <link name="$(arg robot_name)/fingers_link">
+      <link name="$(arg arm_name)/fingers_link">
         <inertial>
           <mass value="0.001" />
@@ -474,12 +474,12 @@
             xyz="0 0 0" />
           <parent
-            link="$(arg robot_name)/fingers_link" />
+            link="$(arg arm_name)/fingers_link" />
           <child
-            link="$(arg robot_name)/left_finger_link" />
+            link="$(arg arm_name)/left_finger_link" />
           <dynamics
             friction="0.1"
             damping="0.1" />
         </joint>
-        <link name="$(arg robot_name)/left_finger_link">
+        <link name="$(arg arm_name)/left_finger_link">
           <visual>
             <origin
@@ -528,7 +528,7 @@
             xyz="0 0 0" />
           <parent
-            link="$(arg robot_name)/fingers_link" />
+            link="$(arg arm_name)/fingers_link" />
           <child
-            link="$(arg robot_name)/right_finger_link" />
+            link="$(arg arm_name)/right_finger_link" />
           <dynamics
             friction="0.1"
@@ -541,5 +541,5 @@
           </xacro:if>
         </joint>
-        <link name="$(arg robot_name)/right_finger_link">
+        <link name="$(arg arm_name)/right_finger_link">
           <visual>
             <origin
@@ -583,9 +583,9 @@
             xyz="0.027575 0 0" />
           <parent
-            link="$(arg robot_name)/fingers_link" />
+            link="$(arg arm_name)/fingers_link" />
           <child
-            link="$(arg robot_name)/ee_gripper_link" />
+            link="$(arg arm_name)/ee_gripper_link" />
         </joint>
-        <link name="$(arg robot_name)/ee_gripper_link">
+        <link name="$(arg arm_name)/ee_gripper_link">
           <inertial>
             <mass value="0.001" />
