Commit message: feat: updated swarmie.urdf.xacro and mariam_rsp.launch.py to flip the camera when the robot name is monica

File: src/mariam_description/xacro_models/swarmie.urdf.xacro (robot description, xacro)
@@ -17,4 +17,13 @@
   <!-- Position the wheels along the x-axis -->
   <xacro:property name="wheel_xoff" value="0.09"/>
+  <!-- Defines the position and orientation of the camera joint -->
+  <!-- if the robot name arg is 'monica', the camera will be flipped by pi radians -->
+  <xacro:macro name="camera_joint" params="robot_name">
+    <joint name="camera_joint" type="fixed">
+      <parent link="base_link"/>
+      <child link="camera_link"/>
+      <origin xyz="-${base_length/2 + 0.01} 0 0.3" rpy="0 0 ${pi if robot_name == 'monica' else 0}"/>
+    </joint>
+  </xacro:macro>
   <!-- Define intertial property macros  -->
   <xacro:macro name="box_inertia" params="m w h d">
@@ -155,8 +164,4 @@
     <xacro:box_inertia m="1.0" w="0.029" d="0.124" h="0.027"/>
   </link>
-  <joint name="camera_joint" type="fixed">
-    <parent link="base_link"/>
-    <child link="camera_link"/>
-    <origin xyz="-${base_length/2 + 0.01} 0 0.3" rpy="0 0 0"/>
-  </joint>
+  <xacro:camera_joint robot_name="$(arg robot_name)"/>
 </robot>

Commit message: update: added vicon link

File: src/mariam_description/xacro_models/swarmie.urdf.xacro (robot description, xacro)
@@ -47,4 +47,11 @@
     </inertial>
   </xacro:macro>
+  <!-- ****************** VICON FRAME ***************************  -->
+  <link name="vicon_link"></link>
+  <joint name="vicon_joint" type="fixed">
+    <parent link="vicon_link"/>
+    <child link="base_link" />
+    <origin xyz="0.1 -0.1 -0.09" rpy="0 0 0"/>
+  </joint>
   <!-- ****************** ROBOT BASE FOOTPRINT ***************************  -->
   <!-- Define the center of the main robot chassis projected on the ground -->

Commit message: fix: removed base_footprint

File: src/mariam_description/xacro_models/swarmie.urdf.xacro (robot description, xacro)
@@ -56,12 +56,11 @@
   <!-- ****************** ROBOT BASE FOOTPRINT ***************************  -->
   <!-- Define the center of the main robot chassis projected on the ground -->
-  <link name="base_footprint">
-  </link>
+  <!-- <link name="base_footprint"></link> -->
   <!-- The base footprint of the robot is located underneath the chassis -->
-  <joint name="base_joint" type="fixed">
-    <parent link="base_footprint"/>
-    <child link="base_link" />
-    <origin xyz="0.0 0.0 ${(wheel_radius+wheel_zoff)}" rpy="0 0 0"/>
-  </joint>
+  <!-- <joint name="base_joint" type="fixed"> -->
+    <!-- <parent link="base_footprint"/> -->
+    <!-- <child link="base_link" /> -->
+    <!-- <origin xyz="0.0 0.0 ${(wheel_radius+wheel_zoff)}" rpy="0 0 0"/> -->
+  <!-- </joint> -->
   <!-- ********************** ROBOT CHASSIS *********************************  -->
   <link name="base_link">
